Commit message: xacro urdf launch on rviz and gazebo

File: src/generic_missile_description/urdf/fins_group.xacro (robot description, xacro)
@@ -16,5 +16,5 @@
         </collision>
         <xacro:inertial_box mass="${finhold_mass}" x="${finhold_height}" y="${wing_thickness}" z="${fin_wide}">
-            <origin xyz="${finhold_height/2} 0 0" rpy="0 0 0"/>
+            <origin xyz="${finhold_height/2} 0 ${fin_wide/2}" rpy="0 0 0"/>
         </xacro:inertial_box>
     </xacro:macro>
@@ -35,5 +35,5 @@
         </collision>
         <xacro:inertial_box mass="${fin_mass}" x="${fin_height}" y="${wing_thickness}" z="${fin_wide}">
-            <origin xyz="${fin_height/2} 0 0" rpy="0 0 0"/>
+            <origin xyz="${fin_height/2} 0 ${fin_wide/2}" rpy="0 0 0"/>
         </xacro:inertial_box>
     </xacro:macro>
@@ -49,7 +49,4 @@
         <xacro:finhold_body_desc />
     </link>/>
-    <gazebo reference="finhold_1">
-        <material>Gazebo/Red</material>
-    </gazebo>
     <!-- 2nd fin holder -->
     <joint name="finhold_2_joint" type="revolute">
@@ -63,7 +60,4 @@
         <xacro:finhold_body_desc />
     </link>/>
-    <gazebo reference="finhold_2">
-        <material>Gazebo/Red</material>
-    </gazebo>
     <!-- 3rd fin holder -->
     <joint name="finhold_3_joint" type="revolute">
@@ -77,7 +71,4 @@
         <xacro:finhold_body_desc />
     </link>/>
-    <gazebo reference="finhold_3">
-        <material>Gazebo/Red</material>
-    </gazebo>
     <!-- 2nd fin holder -->
     <joint name="finhold_4_joint" type="revolute">
@@ -91,7 +82,4 @@
         <xacro:finhold_body_desc />
     </link>/>
-    <gazebo reference="finhold_4">
-        <material>Gazebo/Red</material>
-    </gazebo>
     <!-- 1st fin -->
     <joint name="fin_1_joint" type="revolute">
@@ -105,7 +93,4 @@
         <xacro:fin_body_desc />
     </link>
-    <gazebo reference="fin_1">
-        <material>Gazebo/Red</material>
-    </gazebo>
     <!-- 2nd fin -->
     <joint name="fin_2_joint" type="revolute">
@@ -119,7 +104,4 @@
         <xacro:fin_body_desc />
     </link>
-    <gazebo reference="fin_2">
-        <material>Gazebo/Red</material>
-    </gazebo>
     <!-- 3rd fin -->
     <joint name="fin_3_joint" type="revolute">
@@ -133,7 +115,4 @@
         <xacro:fin_body_desc />
     </link>
-    <gazebo reference="fin_3">
-        <material>Gazebo/Red</material>
-    </gazebo>
     <!-- 4th fin -->
     <joint name="fin_4_joint" type="revolute">
@@ -147,6 +126,3 @@
         <xacro:fin_body_desc />
     </link>
-    <gazebo reference="fin_4">
-        <material>Gazebo/Red</material>
-    </gazebo>
 </robot>

File: src/generic_missile_description/urdf/generic_missile.urdf.xacro (robot description, xacro)
@@ -1,3 +1,6 @@
 <robot xmlns:xacro="http://www.ros.org/wiki/xacro" name="generic_missile">
-    <xacro:include filename="missile_core.xacro" />
+    <xacro:include filename="$(find generic_missile_description)/urdf/missile_core.xacro" />
+    <xacro:include filename="$(find generic_missile_description)/urdf/control_missile.xacro"/>
+    <xacro:include filename="$(find generic_missile_description)/gazebo/physical_missile.gazebo.xacro"/>
+    <!-- <xacro:include filename="$(find generic_missile_description)/gazebo/plugins_missile.gazebo.xacro"/> -->
 </robot>

File: src/generic_missile_description/urdf/missile_core.xacro (robot description, xacro)
@@ -4,12 +4,11 @@
     <xacro:include filename="missile_properties.xacro"/>
     <!-- base link -->
-    <link name="base_link"/>
+    <!-- <link name="base_link"/> -->
     <!-- missile main body -->
-    <joint name="missile_joint" type="fixed">
+    <!-- <joint name="missile_joint" type="fixed">
         <parent link="base_link"/>
         <child link="missile_body"/>
-        <!-- <origin xyz="0 0 1.5" rpy="0 0 0"/> -->
-        <!-- <axis xyz="0 0 0"/> -->
-    </joint>
+        <origin xyz="0 0 0" rpy="0 0 0" />
+    </joint> -->
     <link name="missile_body">
         <visual>
@@ -27,10 +26,7 @@
         </collision>
         <xacro:inertial_cylinder mass="1.0" length="${missile_length}" radius="${missile_radius}">
-            <origin xyz="${missile_length/2} 0 0" rpy="0 ${pi/2} 0"/>
+            <origin xyz="0 0 0" rpy="0 0 0"/>
         </xacro:inertial_cylinder>
     </link>
-    <gazebo reference="missile_body">
-        <material>Gazebo/White</material>
-    </gazebo>
     <!-- head missile -->
     <joint name="head_joint" type="fixed">
@@ -57,4 +53,4 @@
     </link>
     <xacro:include filename="wings_group.xacro"/>
-    <xacro:include filename="fins_group.xacro"/>
+    <!-- <xacro:include filename="fins_group.xacro"/> -->
 </robot>

File: src/generic_missile_description/urdf/missile_properties.xacro (robot description, xacro)
@@ -9,9 +9,9 @@
     <xacro:property name="fin_wide" value="0.3" />
     <xacro:property name="fin_height" value="0.2" />
-    <xacro:property name="fin_mass" value="0.1" />
-    <xacro:property name="finhold_mass" value="0.05" />
+    <xacro:property name="fin_mass" value="0.001" />
+    <xacro:property name="finhold_mass" value="0.3" />
     <xacro:property name="wing_mass" value="0.3" />
     <xacro:property name="body_mass" value="1" />
-    <xacro:property name="head_mass" value="0.2" />
+    <xacro:property name="head_mass" value="0.001" />
     <material name="white">
         <color rgba="1 1 1 1" />

File: src/generic_missile_description/urdf/wings_group.xacro (robot description, xacro)
@@ -16,5 +16,5 @@
         </collision>
         <xacro:inertial_box mass="${wing_mass}" x="${wing_height}" y="${wing_thickness}" z="${wing_thickness}">
-            <origin xyz="${wing_height/2} 0 0" rpy="0 0 0"/>
+            <origin xyz="${wing_height/2} 0 ${wing_wide/2}" rpy="0 0 0"/>
         </xacro:inertial_box>
     </xacro:macro>
@@ -30,9 +30,6 @@
         <xacro:wing_body_desc />
     </link>/>
-    <gazebo reference="wing_1">
-        <material>Gazebo/Red</material>
-    </gazebo>
     <!-- 2nd wing -->
-    <joint name="wing_2_joint" type="revolute">
+    <!-- <joint name="wing_2_joint" type="revolute">
         <parent link="missile_body"/>
         <child link="wing_2"/>
@@ -43,10 +40,7 @@
     <link name="wing_2">
         <xacro:wing_body_desc />
-    </link>/>
-    <gazebo reference="wing_2">
-        <material>Gazebo/Red</material>
-    </gazebo>
+    </link>/> -->
     <!-- 3rd wing -->
-    <joint name="wing_3_joint" type="revolute">
+    <!-- <joint name="wing_3_joint" type="revolute">
         <parent link="missile_body"/>
         <child link="wing_3"/>
@@ -57,10 +51,7 @@
     <link name="wing_3">
         <xacro:wing_body_desc />
-    </link>/>
-    <gazebo reference="wing_3">
-        <material>Gazebo/Red</material>
-    </gazebo>
+    </link>/> -->
     <!-- 4th wing -->
-    <joint name="wing_4_joint" type="revolute">
+    <!-- <joint name="wing_4_joint" type="revolute">
         <parent link="missile_body"/>
         <child link="wing_4"/>
@@ -71,7 +62,4 @@
     <link name="wing_4">
         <xacro:wing_body_desc />
-    </link>/>
-    <gazebo reference="wing_4">
-        <material>Gazebo/Red</material>
-    </gazebo>
+    </link>/> -->
 </robot>
