Commit message: try the forward position controller

File: src/generic_missile_description/urdf/control_missile.xacro (robot description, xacro)
@@ -1,9 +1,6 @@
 <?xml version="1.0"?>
 <robot xmlns:xacro="http://www.ros.org/wiki/xacro">
-    <ros2_control name="GazeboSystem" type="sysetem">
-        <hardware>
-            <plugin>gazebo_ros2_control/GazeboSystem</plugin>
-        </hardware>
-        <joint name="wing_1_joint" >
+    <xacro:macro name="wings_joint" params="joint_name">
+        <joint name="${joint_name}" >
             <command_interface name="position">
                 <param name="min">-1000</param>
@@ -12,6 +9,22 @@
             <state_interface name="position"/>
             <state_interface name="velocity"/>
-            <state_interface name="effort"/>
         </joint>
+    </xacro:macro>
+    <ros2_control name="GazeboSystem" type="sysetem">
+        <hardware>
+            <plugin>gazebo_ros2_control/GazeboSystem</plugin>
+        </hardware>
+        <xacro:wings_joint joint_name="wing_1_joint"/>
+        <xacro:wings_joint joint_name="wing_2_joint"/>
+        <xacro:wings_joint joint_name="wing_3_joint"/>
+        <xacro:wings_joint joint_name="wing_4_joint"/>
+        <!-- <joint name="wing_1_joint" >
+            <command_interface name="position">
+                <param name="min">${-pi*2/3}</param>
+                <param name="max">${pi*2/3}</param>
+            </command_interface>
+            <state_interface name="position"/>
+            <state_interface name="velocity"/>
+        </joint> -->
     </ros2_control>
     <gazebo>

File: src/generic_missile_description/urdf/generic_missile.urdf.xacro (robot description, xacro)
@@ -1,6 +1,6 @@
 <robot xmlns:xacro="http://www.ros.org/wiki/xacro" name="generic_missile">
     <xacro:include filename="$(find generic_missile_description)/urdf/missile_core.xacro" />
+    <xacro:include filename="$(find generic_missile_description)/gazebo/physical_missile.gazebo.xacro"/>
     <xacro:include filename="$(find generic_missile_description)/urdf/control_missile.xacro"/>
-    <xacro:include filename="$(find generic_missile_description)/gazebo/physical_missile.gazebo.xacro"/>
     <!-- <xacro:include filename="$(find generic_missile_description)/gazebo/plugins_missile.gazebo.xacro"/> -->
 </robot>

File: src/generic_missile_description/urdf/missile_core.xacro (robot description, xacro)
@@ -3,12 +3,16 @@
     <xacro:include filename="inertial_macros.xacro"/>
     <xacro:include filename="missile_properties.xacro"/>
+    <link name="world"/>
+    <gazebo reference="world">
+      <static>true</static>
+    </gazebo>
     <!-- base link -->
     <!-- <link name="base_link"/> -->
     <!-- missile main body -->
-    <!-- <joint name="missile_joint" type="fixed">
-        <parent link="base_link"/>
+    <joint name="missile_joint" type="fixed">
+        <parent link="world"/>
         <child link="missile_body"/>
         <origin xyz="0 0 0" rpy="0 0 0" />
-    </joint> -->
+    </joint>
     <link name="missile_body">
         <visual>

File: src/generic_missile_description/urdf/missile_properties.xacro (robot description, xacro)
@@ -11,7 +11,7 @@
     <xacro:property name="fin_mass" value="0.001" />
     <xacro:property name="finhold_mass" value="0.3" />
-    <xacro:property name="wing_mass" value="0.3" />
-    <xacro:property name="body_mass" value="1" />
-    <xacro:property name="head_mass" value="0.001" />
+    <xacro:property name="wing_mass" value="0.1" />
+    <xacro:property name="body_mass" value="1.5" />
+    <xacro:property name="head_mass" value="0.2" />
     <material name="white">
         <color rgba="1 1 1 1" />

File: src/generic_missile_description/urdf/wings_group.xacro (robot description, xacro)
@@ -31,5 +31,5 @@
     </link>/>
     <!-- 2nd wing -->
-    <!-- <joint name="wing_2_joint" type="revolute">
+    <joint name="wing_2_joint" type="revolute">
         <parent link="missile_body"/>
         <child link="wing_2"/>
@@ -40,7 +40,7 @@
     <link name="wing_2">
         <xacro:wing_body_desc />
-    </link>/> -->
+    </link>/>
     <!-- 3rd wing -->
-    <!-- <joint name="wing_3_joint" type="revolute">
+    <joint name="wing_3_joint" type="revolute">
         <parent link="missile_body"/>
         <child link="wing_3"/>
@@ -51,7 +51,7 @@
     <link name="wing_3">
         <xacro:wing_body_desc />
-    </link>/> -->
+    </link>/>
     <!-- 4th wing -->
-    <!-- <joint name="wing_4_joint" type="revolute">
+    <joint name="wing_4_joint" type="revolute">
         <parent link="missile_body"/>
         <child link="wing_4"/>
@@ -62,4 +62,4 @@
     <link name="wing_4">
         <xacro:wing_body_desc />
-    </link>/> -->
+    </link>/>
 </robot>
